File: 4056M.kicad_sch (KiCad schematic)
At the start: 25 parts, among them J1 VBUS, J2 GND, J3 Conn_01x02_MountingPin, J4 3V3, J5 state, J6 measure, Q1 3401, Q2 8050, Q3 3401, U1 TC4056A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

Commit message: 电池座PIN1应该为GND
Connections:
- net +BATT: now also J3.2 (Pin_2); no longer J3.1 (Pin_1)
- net -BATT: now also J3.1 (Pin_1); no longer J3.2 (Pin_2)
Changed lines of the file:
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@@
 (kicad_sch (version 20211123) (generator eeschema)
   (paper "A4")
+  (junction (at 92.71 101.854) (diameter 0) (color 0 0 0 0)
+  )
   (junction (at 32.258 85.09) (diameter 0) (color 0 0 0 0)
   )
   (junction (at 138.176 105.664) (diameter 0) (color 0 0 0 0)
   )
-  (junction (at 92.202 104.394) (diameter 0) (color 0 0 0 0)
-  )
   (junction (at 218.44 83.82) (diameter 0) (color 0 0 0 0)
   )
-  (junction (at 92.202 101.854) (diameter 0) (color 0 0 0 0)
-  )
   (junction (at 129.286 95.504) (diameter 0) (color 0 0 0 0)
   )
@@
   (junction (at 218.44 100.33) (diameter 0) (color 0 0 0 0)
   )
+  (junction (at 92.71 104.394) (diameter 0) (color 0 0 0 0)
+  )
   (junction (at 66.548 87.122) (diameter 0) (color 0 0 0 0)
   )
@@
     (stroke (width 0) (type default) (color 0 0 0 0))
   )
-  (wire (pts (xy 92.202 101.854) (xy 94.742 101.854))
+  (wire (pts (xy 89.662 104.394) (xy 92.71 104.394))
     (stroke (width 0) (type default) (color 0 0 0 0))
   )
@@
     (stroke (width 0) (type default) (color 0 0 0 0))
   )
-  (wire (pts (xy 92.202 104.394) (xy 94.742 104.394))
-    (stroke (width 0) (type default) (color 0 0 0 0))
-  )
   (wire (pts (xy 76.073 87.122) (xy 79.248 87.122))
     (stroke (width 0) (type default) (color 0 0 0 0))
@@
     (stroke (width 0) (type default) (color 0 0 0 0))
   )
-  (wire (pts (xy 92.202 104.394) (xy 92.202 105.664))
-    (stroke (width 0) (type default) (color 0 0 0 0))
-  )
   (wire (pts (xy 209.55 99.06) (xy 209.55 100.33))
     (stroke (width 0) (type default) (color 0 0 0 0))
   )
-  (wire (pts (xy 89.662 101.854) (xy 92.202 101.854))
+  (wire (pts (xy 92.71 100.33) (xy 92.71 101.854))
     (stroke (width 0) (type default) (color 0 0 0 0))
   )
@@
     (stroke (width 0) (type default) (color 0 0 0 0))
   )
+  (wire (pts (xy 92.71 101.854) (xy 95.504 101.854))
+    (stroke (width 0) (type default) (color 0 0 0 0))
+  )
   (wire (pts (xy 209.55 88.9) (xy 210.82 88.9))
     (stroke (width 0) (type default) (color 0 0 0 0))
@@
     (stroke (width 0) (type default) (color 0 0 0 0))
   )
+  (wire (pts (xy 92.71 104.394) (xy 95.504 104.394))
+    (stroke (width 0) (type default) (color 0 0 0 0))
+  )
   (wire (pts (xy 209.55 88.9) (xy 209.55 91.44))
     (stroke (width 0) (type default) (color 0 0 0 0))
@@
     (stroke (width 0) (type default) (color 0 0 0 0))
   )
-  (wire (pts (xy 92.202 100.838) (xy 92.202 101.854))
-    (stroke (width 0) (type default) (color 0 0 0 0))
-  )
   (wire (pts (xy 32.258 97.79) (xy 32.258 100.33))
     (stroke (width 0) (type default) (color 0 0 0 0))
@@
     (stroke (width 0) (type default) (color 0 0 0 0))
   )
+  (wire (pts (xy 92.71 104.394) (xy 92.71 106.172))
+    (stroke (width 0) (type default) (color 0 0 0 0))
+  )
   (wire (pts (xy 227.33 96.52) (xy 227.33 97.155))
     (stroke (width 0) (type default) (color 0 0 0 0))
@@
     (stroke (width 0) (type default) (color 0 0 0 0))
   )
-  (wire (pts (xy 89.662 104.394) (xy 92.202 104.394))
-    (stroke (width 0) (type default) (color 0 0 0 0))
-  )
   (wire (pts (xy 27.178 97.79) (xy 32.258 97.79))
     (stroke (width 0) (type default) (color 0 0 0 0))
@@
   )
   (wire (pts (xy 68.453 87.122) (xy 66.548 87.122))
+    (stroke (width 0) (type default) (color 0 0 0 0))
+  )
+  (wire (pts (xy 89.662 101.854) (xy 92.71 101.854))
     (stroke (width 0) (type default) (color 0 0 0 0))
   )
@@
     (pin "2")
   )
-  (symbol (lib_id "power:GND") (at 92.202 105.664 0) (unit 1)
-    (in_bom yes) (on_board yes) (fields_autoplaced)
-    (property "Reference" "#PWR08" (id 0) (at 92.202 112.014 0)
-      (effects (font (size 1.27 1.27)) hide)
-    )
-    (property "Value" "GND" (id 1) (at 92.202 110.998 0))
-    (property "Footprint" "" (id 2) (at 92.202 105.664 0)
-      (effects (font (size 1.27 1.27)) hide)
-    )
-    (property "Datasheet" "" (id 3) (at 92.202 105.664 0)
+  (symbol (lib_id "power:GND") (at 92.71 100.33 180) (unit 1)
+    (in_bom yes) (on_board yes) (fields_autoplaced)
+    (property "Reference" "#PWR08" (id 0) (at 92.71 93.98 0)
+      (effects (font (size 1.27 1.27)) hide)
+    )
+    (property "Value" "GND" (id 1) (at 92.71 94.996 0))
+    (property "Footprint" "" (id 2) (at 92.71 100.33 0)
+      (effects (font (size 1.27 1.27)) hide)
+    )
+    (property "Datasheet" "" (id 3) (at 92.71 100.33 0)
       (effects (font (size 1.27 1.27)) hide)
     )
@@
     (pin "1")
   )
-  (symbol (lib_id "power:-BATT") (at 94.742 104.394 270) (unit 1)
-    (in_bom yes) (on_board yes) (fields_autoplaced)
-    (property "Reference" "#PWR09" (id 0) (at 90.932 104.394 0)
-      (effects (font (size 1.27 1.27)) hide)
-    )
-    (property "Value" "-BATT" (id 1) (at 99.06 104.3939 90)
-      (effects (font (size 1.27 1.27)) (justify left))
-    )
-    (property "Footprint" "" (id 2) (at 94.742 104.394 0)
-      (effects (font (size 1.27 1.27)) hide)
-    )
-    (property "Datasheet" "" (id 3) (at 94.742 104.394 0)
+  (symbol (lib_id "power:-BATT") (at 95.504 101.854 270) (unit 1)
+    (in_bom yes) (on_board yes) (fields_autoplaced)
+    (property "Reference" "#PWR09" (id 0) (at 91.694 101.854 0)
+      (effects (font (size 1.27 1.27)) hide)
+    )
+    (property "Value" "-BATT" (id 1) (at 99.822 101.8539 90)
+      (effects (font (size 1.27 1.27)) (justify left))
+    )
+    (property "Footprint" "" (id 2) (at 95.504 101.854 0)
+      (effects (font (size 1.27 1.27)) hide)
+    )
+    (property "Datasheet" "" (id 3) (at 95.504 101.854 0)
       (effects (font (size 1.27 1.27)) hide)
     )
@@
     (pin "1")
   )
-  (symbol (lib_id "power:PWR_FLAG") (at 92.202 100.838 0) (unit 1)
-    (in_bom yes) (on_board yes) (fields_autoplaced)
-    (property "Reference" "#FLG03" (id 0) (at 92.202 98.933 0)
-      (effects (font (size 1.27 1.27)) hide)
-    )
-    (property "Value" "PWR_FLAG" (id 1) (at 92.202 96.266 0))
-    (property "Footprint" "" (id 2) (at 92.202 100.838 0)
-      (effects (font (size 1.27 1.27)) hide)
-    )
-    (property "Datasheet" "~" (id 3) (at 92.202 100.838 0)
+  (symbol (lib_id "power:PWR_FLAG") (at 92.71 106.172 180) (unit 1)
+    (in_bom yes) (on_board yes) (fields_autoplaced)
+    (property "Reference" "#FLG03" (id 0) (at 92.71 108.077 0)
+      (effects (font (size 1.27 1.27)) hide)
+    )
+    (property "Value" "PWR_FLAG" (id 1) (at 92.71 110.998 0))
+    (property "Footprint" "" (id 2) (at 92.71 106.172 0)
+      (effects (font (size 1.27 1.27)) hide)
+    )
+    (property "Datasheet" "~" (id 3) (at 92.71 106.172 0)
       (effects (font (size 1.27 1.27)) hide)
     )
@@
     (pin "2")
   )
-  (symbol (lib_id "power:+BATT") (at 94.742 101.854 270) (unit 1)
-    (in_bom yes) (on_board yes) (fields_autoplaced)
-    (property "Reference" "#PWR010" (id 0) (at 90.932 101.854 0)
-      (effects (font (size 1.27 1.27)) hide)
-    )
-    (property "Value" "+BATT" (id 1) (at 99.06 101.8539 90)
-      (effects (font (size 1.27 1.27)) (justify left))
-    )
-    (property "Footprint" "" (id 2) (at 94.742 101.854 0)
-      (effects (font (size 1.27 1.27)) hide)
-    )
-    (property "Datasheet" "" (id 3) (at 94.742 101.854 0)
-      (effects (font (size 1.27 1.27)) hide)
-    )
+  (symbol (lib_id "power:+BATT") (at 95.504 104.394 270) (unit 1)
+    (in_bom yes) (on_board yes) (fields_autoplaced)
+    (property "Reference" "#PWR010" (id 0) (at 91.694 104.394 0)
+      (effects (font (size 1.27 1.27)) hide)
+    )
+    (property "Value" "+BATT" (id 1) (at 99.822 104.3939 90)
+      (effects (font (size 1.27 1.27)) (justify left))
+    )
+    (property "Footprint" "" (id 2) (at 95.504 104.394 0)
+      (effects (font (size 1.27 1.27)) hide)
+    )
+    (property "Datasheet" "" (id 3) (at 95.504 104.394 0)
+      (effects (font (size 1.27 1.27)) hide)
+    )

Commit message: New version
Parts:
- removed J6: measure, Connector_PinHeader_1.27mm:PinHeader_1x02_P1.27mm_Vertical, symbol Connector_Generic:Conn_01x02
- removed Q2: 8050, Package_TO_SOT_SMD:SOT-23, symbol Device:Q_NPN_BEC
- removed Q3: 3401, Package_TO_SOT_SMD:SOT-23, symbol Device:Q_PMOS_GSD
- removed R7: 4.7K, Resistor_SMD:R_0603_1608Metric, symbol Device:R
- removed R8: 1K, Resistor_SMD:R_0603_1608Metric, symbol Device:R
- removed U1: TC4056A, Package_SO:HSOP-8-1EP_3.9x4.9mm_P1.27mm_EP2.3x2.3mm, symbol 4056M:TC4056A
- added C5, C6: 1uF, Capacitor_SMD:C_0603_1608Metric, symbol Device:C
- added J6: Conn_01x04, Connector_PinHeader_1.27mm:PinHeader_1x04_P1.27mm_Vertical, symbol Connector_Generic:Conn_01x04
- added U1: TP4057, Package_TO_SOT_SMD:SOT-23-6, symbol 4056M:TP4057
- added U4: CW2015, Package_DFN_QFN:TDFN-8-1EP_3x2mm_P0.5mm_EP1.4x1.4mm, symbol 4056M:CW2015
- C2: footprint Capacitor_SMD:C_1206_3216Metric -> Capacitor_SMD:C_0603_1608Metric
- R2: footprint Resistor_SMD:R_0603_1608Metric -> Resistor_SMD:R_0402_1005Metric
- R4: value 1K -> 470R
- R5: value 100K -> 100R
- R6: value 10K -> 4.7K
Connections:
- net IO is gone; now on net +BATT: R4.1
- net +BATT: now also R5.1, U1.3 (BAT); no longer R6.1
- net -BATT: now also C5.1, C6.2, U1.2 (GND), U4.1 (CTG), U4.4 (GND), U4.6 (QSTRT), U4.9 (EP); no longer R5.2
- net CHRG: now also J5.2 (Pin_2), U1.1 (CHRG); no longer J5.1 (Pin_1)
- net STDBY: now also J5.1 (Pin_1), U1.5 (STDBY); no longer J5.2 (Pin_2)
- net VBUS: now also U1.4 (VCC)
- net at R4.2: now also C5.2, U4.2 (CELL); no longer R5.1
- net ALRT: now reaches R6.2
- net ALRT: now also J6.2 (Pin_2), U4.5 (ALRT)
- net at R1.2: now also U1.6 (PROG)
- new net: C6.1, R5.2, U4.3 (VDD)
- new net PS: J6.1 (Pin_1), R6.1
- new net SCL: J6.3 (Pin_3), U4.7 (SCL)
- new net SDA: J6.4 (Pin_4), U4.8 (SDA)
Other:
- moved on the sheet: R1
